Commit message: hardware interface

File: src/dd_bot/description/robot.urdf.xacro (robot description, xacro)
@@ -4,5 +4,4 @@
     <xacro:arg name="sim_mode" default="false"/>
     <xacro:include filename="robot_core.xacro" />
-    <xacro:include filename="gazebo_control.xacro" />
     <xacro:include filename="lidar.xacro" />
     <xacro:include filename="left_camera.xacro" />

File: src/dd_bot/description/robot_core.xacro (robot description, xacro)
@@ -73,30 +73,4 @@
         <material>Gazebo/White</material>
     </gazebo>
-<!-- right wheel link-->
-    <joint name="right_wheel_joint" type="continuous">
-        <parent link="base_link"/>
-        <child link="right_wheel"/>
-        <origin xyz="0.0 0.28 0.02" rpy="-${pi/2} 0.0 0.0"/>
-        <axis xyz="0.0 0.0 1"/>
-    </joint>
-    <link name="right_wheel">
-        <visual>
-            <geometry>
-                <cylinder radius="0.1" length="0.04"/>
-            </geometry>
-            <material name="blue"/>
-        </visual>
-        <collision>
-            <geometry>
-                <cylinder radius="0.1" length="0.04"/>
-            </geometry>
-        </collision>
-        <xacro:inertial_cylinder mass="0.1" length="0.04" radius="0.1" >
-            <origin xyz="0.0 0.0 0.0" rpy="0.0 0.0 0.0"/>
-        </xacro:inertial_cylinder>
-    </link>
-    <gazebo reference="right_wheel">
-        <material>Gazebo/Blue</material>
-    </gazebo>
 <!-- left wheel link-->
     <joint name="left_wheel_joint" type="continuous">
@@ -123,4 +97,30 @@
     </link>
     <gazebo reference="left_wheel">
+        <material>Gazebo/Blue</material>
+    </gazebo>
+<!-- right wheel link-->
+    <joint name="right_wheel_joint" type="continuous">
+        <parent link="base_link"/>
+        <child link="right_wheel"/>
+        <origin xyz="0.0 0.28 0.02" rpy="${-pi/2} 0.0 0.0"/>
+        <axis xyz="0 0 -1"/>
+    </joint>
+    <link name="right_wheel">
+        <visual>
+            <geometry>
+                <cylinder radius="0.1" length="0.04"/>
+            </geometry>
+            <material name="blue"/>
+        </visual>
+        <collision>
+            <geometry>
+                <cylinder radius="0.1" length="0.04"/>
+            </geometry>
+        </collision>
+        <xacro:inertial_cylinder mass="0.1" length="0.04" radius="0.1" >
+            <origin xyz="0.0 0.0 0.0" rpy="0.0 0.0 0.0"/>
+        </xacro:inertial_cylinder>
+    </link>
+    <gazebo reference="right_wheel">
         <material>Gazebo/Blue</material>
     </gazebo>

File: src/dd_bot/description/ros2_control.xacro (robot description, xacro)
@@ -1,5 +1,5 @@
 <?xml version="1.0"?>
 <robot xmlns:xacro="http://www.ros.org/wiki/xacro">
-    <!-- <xacro:unless value="$(arg sim_mode)">
+    <!-- <xacro:unless value="$(arg sim_mode)"> -->
         <ros2_control name="RealRobot" type="system">
             <hardware>
@@ -30,7 +30,7 @@
             </joint>
         </ros2_control>
-    </xacro:unless> -->
+    <!-- </xacro:unless> -->
     <!-- <xacro:if value="$(arg sim_mode)"> -->
-    <ros2_control name="GazeboSystem" type="system">
+    <!-- <ros2_control name="GazeboSystem" type="system">
         <hardware>
             <plugin>gz_ros2_control/GazeboSimSystem</plugin>
@@ -52,11 +52,11 @@
             <state_interface name="position"/>
         </joint>
-    </ros2_control>
+    </ros2_control> -->
     <!-- </xacro:if> -->
-    <gazebo>
+    <!-- <gazebo>
         <plugin name="gz_ros2_control::GazeboSimROS2ControlPlugin" filename="libgz_ros2_control-system.so">
             <parameters>$(find dd_bot)/config/my_controllers.yaml</parameters>
-            <!-- <parameters>$(find dd_bot)/config/gaz_ros2_ctl_use_sim.yaml</parameters> -->
+            <parameters>$(find dd_bot)/config/gaz_ros2_ctl_use_sim.yaml</parameters>
         </plugin>
-    </gazebo>
+    </gazebo> -->
 </robot>
