Commit message: lidar fix

File: src/dd_bot/description/lidar.xacro (robot description, xacro)
@@ -4,5 +4,5 @@
         <parent link="base_link"/>
         <child link="laser_frame"/>
-        <origin xyz="0.0 0.125 0.26" rpy="0 0 0"/>
+        <origin xyz="0.0 0.125 0.26" rpy="0 0 ${pi}"/>
     </joint>
     <link name="laser_frame">

File: src/dd_bot/description/robot_core.xacro (robot description, xacro)
@@ -17,4 +17,13 @@
     <link name="base_link">
     </link>
+<!-- Base_Footprint link-->
+    <joint name="base_footprint_joint" type="fixed">
+        <parent link="base_link"/>
+        <child link="base_footprint"/>
+        <origin xyz="0 0 0" rpy="0 0 0"/>
+    </joint>
+    <link name="base_footprint">
+    </link>
+<!-- chasis link-->
     <joint name="chassis_joint" type="fixed">
         <parent link="base_link"/>
@@ -22,5 +31,4 @@
         <origin xyz="0.045 0 0"/>
     </joint>
-<!-- chasis link-->
     <link name="chassis">
         <visual>

File: src/dd_bot/description/ros2_control.xacro (robot description, xacro)
@@ -57,5 +57,5 @@
         <plugin name="gz_ros2_control::GazeboSimROS2ControlPlugin" filename="libgz_ros2_control-system.so">
             <parameters>$(find dd_bot)/config/my_controllers.yaml</parameters>
-            <parameters>$(find dd_bot)/config/gaz_ros2_ctl_use_sim.yaml</parameters>
+            <!-- <parameters>$(find dd_bot)/config/gaz_ros2_ctl_use_sim.yaml</parameters> -->
         </plugin>
     </gazebo>
