Commit message: gazebo and real

File: install/dd_bot/share/dd_bot/description/left_camera.xacro (robot description, xacro)
@@ -14,5 +14,5 @@
         </visual>
         <visual>
-            <origin xyz="-0.01 -0.03 0.0" rpy="0 1.5708 0"/>
+            <origin xyz="0.01 0.03 0.0" rpy="0 1.5708 0"/>
             <geometry>
                 <cylinder radius="0.01" length="0.02"/>
@@ -24,5 +24,5 @@
         <parent link="left_camera_link"/>
         <child link="left_camera_link_optical"/>
-        <origin xyz="0 -0.03 0" rpy="${-pi/2} 0 ${-pi*3/2}"/>
+        <origin xyz="0 0.03 0" rpy="${-pi/2} 0 ${-pi/2}"/>
     </joint>
     <link name="left_camera_link_optical"></link>

File: install/dd_bot/share/dd_bot/description/lidar.xacro (robot description, xacro)
@@ -4,5 +4,5 @@
         <parent link="base_link"/>
         <child link="laser_frame"/>
-        <origin xyz="0.0 -0.125 0.26" rpy="0 0 0"/>
+        <origin xyz="0.0 0.125 0.26" rpy="0 0 0"/>
     </joint>
     <link name="laser_frame">

File: install/dd_bot/share/dd_bot/description/right_camera.xacro (robot description, xacro)
@@ -14,5 +14,5 @@
         </visual>
         <visual>
-            <origin xyz="-0.01 -0.03 0.0" rpy="0 1.5708 0"/>
+            <origin xyz="0.01 -0.03 0.0" rpy="0 1.5708 0"/>
             <geometry>
                 <cylinder radius="0.01" length="0.02"/>
@@ -24,5 +24,5 @@
         <parent link="right_camera_link"/>
         <child link="right_camera_link_optical"/>
-        <origin xyz="0 0.03 0" rpy="${-pi/2} 0 ${-pi*3/2}"/>
+        <origin xyz="0 -0.03 0" rpy="${-pi/2} 0 ${-pi/2}"/>
     </joint>
     <link name="right_camera_link_optical"></link>

File: install/dd_bot/share/dd_bot/description/robot_core.xacro (robot description, xacro)
@@ -20,10 +20,10 @@
         <parent link="base_link"/>
         <child link="chassis"/>
-        <origin xyz="-0.045 0 0"/>
+        <origin xyz="0.045 0 0"/>
     </joint>
 <!-- chasis link-->
     <link name="chassis">
         <visual>
-            <origin xyz="0.045 0.0 0.165" />
+            <origin xyz="-0.045 0.0 0.165" />
             <geometry>
                 <box size="0.19 0.5 0.15"/>
@@ -32,5 +32,5 @@
         </visual>
         <visual>
-            <origin xyz="0.33 0.0 0.10" />
+            <origin xyz="-0.33 0.0 0.10" />
             <geometry>
                 <box size="0.57 0.08 0.02"/>
@@ -39,5 +39,5 @@
         </visual>
         <visual>
-            <origin xyz="0.045 0.0 0.055" />
+            <origin xyz="-0.045 0.0 0.055" />
             <geometry>
                 <box size="0.09 0.5 0.11"/>
@@ -46,17 +46,18 @@
         </visual>
         <collision>
-            <origin xyz="0.045 0.0 0.165" />
+            <origin xyz="-0.045 0.0 0.165" />
             <geometry>
                 <box size="0.19 0.5 0.15"/>
             </geometry>
         </collision>
+        <visual>
+            <origin xyz="-0.33 0.0 0.10" />
+            <geometry>
+                <box size="0.57 0.08 0.02"/>
+            </geometry>
+            <material name="white" />
+        </visual>
         <collision>
-            <origin xyz="0.045 0.0 0.165" />
-            <geometry>
-                <box size="0.19 0.5 0.15"/>
-            </geometry>
-        </collision>
-        <collision>
-            <origin xyz="0.045 0.0 0.055" />
+            <origin xyz="-0.045 0.0 0.055" />
             <geometry>
                 <box size="0.09 0.5 0.11"/>
@@ -64,5 +65,5 @@
         </collision>
         <inertial>
-        <origin xyz="0.20 0.0 0" rpy="0 0 0"/>
+        <origin xyz="-0.20 0.0 0" rpy="0 0 0"/>
         <mass value="1.9809343e+01"/>
         <inertia ixx="4.914e-01" iyy="2.317e-01" izz="5.354e-01"
@@ -73,12 +74,12 @@
         <material>Gazebo/White</material>
     </gazebo>
-<!-- left wheel link-->
-    <joint name="left_wheel_joint" type="continuous">
+<!-- right wheel link-->
+    <joint name="right_wheel_joint" type="continuous">
         <parent link="base_link"/>
-        <child link="left_wheel"/>
+        <child link="right_wheel"/>
         <origin xyz="0 -0.28 0.02" rpy="${pi/2} 0 0"/>
         <axis xyz="0 0 -1"/>
     </joint>
-    <link name="left_wheel">
+    <link name="right_wheel">
         <visual>
             <geometry>
@@ -96,15 +97,15 @@
         </xacro:inertial_cylinder>
     </link>
-    <gazebo reference="left_wheel">
+    <gazebo reference="right_wheel">
         <material>Gazebo/Blue</material>
     </gazebo>
-<!-- right wheel link-->
-    <joint name="right_wheel_joint" type="continuous">
+<!-- left wheel link-->
+    <joint name="left_wheel_joint" type="continuous">
         <parent link="base_link"/>
-        <child link="right_wheel"/>
-        <origin xyz="0.0 0.28 0.02" rpy="${-pi/2} 0.0 0.0"/>
+        <child link="left_wheel"/>
+        <origin xyz="0.0 0.28 0.02" rpy="${-pi/2}  0.0 0.0"/>
         <axis xyz="0 0 1"/>
     </joint>
-    <link name="right_wheel">
+    <link name="left_wheel">
         <visual>
             <geometry>
@@ -122,5 +123,5 @@
         </xacro:inertial_cylinder>
     </link>
-    <gazebo reference="right_wheel">
+    <gazebo reference="left_wheel">
         <material>Gazebo/Blue</material>
     </gazebo>
@@ -129,5 +130,5 @@
         <parent link="chassis"/>
         <child link="caster_wheel"/>
-        <origin xyz="0.6 0 0.00" />
+        <origin xyz="-0.6 0 0.00" />
     </joint>
     <link name="caster_wheel">

File: install/dd_bot/share/dd_bot/description/ros2_control.xacro (robot description, xacro)
@@ -1,5 +1,5 @@
 <?xml version="1.0"?>
 <robot xmlns:xacro="http://www.ros.org/wiki/xacro">
-    <!-- <xacro:unless value="$(arg sim_mode)"> -->
+    <xacro:unless value="$(arg sim_mode)">
         <ros2_control name="RealRobot" type="system">
             <hardware>
@@ -30,33 +30,33 @@
             </joint>
         </ros2_control>
-    <!-- </xacro:unless> -->
-    <!-- <xacro:if value="$(arg sim_mode)"> -->
-    <!-- <ros2_control name="GazeboSystem" type="system">
-        <hardware>
-            <plugin>gz_ros2_control/GazeboSimSystem</plugin>
-        </hardware>
-        <joint name="left_wheel_joint">
-            <command_interface name="velocity">
-                <param name="min">-10</param>
-                <param name="max">10</param>
-            </command_interface>
-            <state_interface name="velocity"/>
-            <state_interface name="position"/>
-        </joint>
-        <joint name="right_wheel_joint">
-            <command_interface name="velocity">
-                <param name="min">-10</param>
-                <param name="max">10</param>
-            </command_interface>
-            <state_interface name="velocity"/>
-            <state_interface name="position"/>
-        </joint>
-    </ros2_control> -->
-    <!-- </xacro:if> -->
-    <!-- <gazebo>
+    </xacro:unless>
+    <xacro:if value="$(arg sim_mode)">
+        <ros2_control name="GazeboSystem" type="system">
+            <hardware>
+                <plugin>gz_ros2_control/GazeboSimSystem</plugin>
+            </hardware>
+            <joint name="left_wheel_joint">
+                <command_interface name="velocity">
+                    <param name="min">-10</param>
+                    <param name="max">10</param>
+                </command_interface>
+                <state_interface name="velocity"/>
+                <state_interface name="position"/>
+            </joint>
+            <joint name="right_wheel_joint">
+                <command_interface name="velocity">
+                    <param name="min">-10</param>
+                    <param name="max">10</param>
+                </command_interface>
+                <state_interface name="velocity"/>
+                <state_interface name="position"/>
+            </joint>
+        </ros2_control>
+    </xacro:if>
+    <gazebo>
         <plugin name="gz_ros2_control::GazeboSimROS2ControlPlugin" filename="libgz_ros2_control-system.so">
             <parameters>$(find dd_bot)/config/my_controllers.yaml</parameters>
             <parameters>$(find dd_bot)/config/gaz_ros2_ctl_use_sim.yaml</parameters>
         </plugin>
-    </gazebo> -->
+    </gazebo>
 </robot>
