Commit message: fyp2 complete

File: src/golftrolley/description/camera.xacro (robot description, xacro)
@@ -1,10 +1,10 @@
 <?xml version="1.0"?>
 <robot xmlns:xacro="http://www.ros.org/wiki/xacro" >
-    <joint name="left_camera_joint" type="fixed">
+    <joint name="camera_joint" type="fixed">
         <parent link="base_link"/>
-        <child link="left_camera_link"/>
-        <origin xyz="0.0 0.0 0.7" rpy="0 0 0"/>
+        <child link="camera_link"/>
+        <origin xyz="0.0 0.0 0.36" rpy="0 0 0"/>
     </joint>
-    <link name="left_camera_link">
+    <link name="camera_link">
         <visual>
             <geometry>
@@ -14,5 +14,5 @@
         </visual>
         <visual>
-            <origin xyz="0.01 0.03 0.0" rpy="0 1.5708 0"/>
+            <origin xyz="0.01 0.0 0.0" rpy="0 1.5708 0"/>
             <geometry>
                 <cylinder radius="0.01" length="0.02"/>
@@ -21,18 +21,18 @@
         </visual>
     </link>
-    <joint name="left_camera_optical_joint" type="fixed">
-        <parent link="left_camera_link"/>
-        <child link="left_camera_link_optical"/>
-        <origin xyz="0 0.03 0" rpy="${-pi/2} 0 ${-pi/2}"/>
+    <joint name="camera_optical_joint" type="fixed">
+        <parent link="camera_link"/>
+        <child link="camera_link_optical"/>
+        <origin xyz="0 0 0" rpy="${-pi/2} 0 ${-pi/2}"/>
     </joint>
-    <link name="left_camera_link_optical"></link>
-    <gazebo reference="left_camera_link">
+    <link name="camera_link_optical"></link>
+    <gazebo reference="camera_link">
         <material>Gazebo/Black</material>
-        <sensor name="left_camera" type="camera">
+        <sensor name="camera" type="camera">
             <pose> 0 0 0 0 0 ${pi} </pose>
             <visualize>true</visualize>
             <update_rate>10</update_rate>
-            <camera name="left_camera">
-                <camera_info_topic>left_camera/camera_info</camera_info_topic>
+            <camera name="camera">
+                <camera_info_topic>camera/camera_info</camera_info_topic>
                 <horizontal_fov>1.089</horizontal_fov>
                 <image>
@@ -46,6 +46,6 @@
                 </clip>
             </camera>
-            <topic>left_camera/image_raw</topic>
-            <gz_frame_id>left_camera_link_optical</gz_frame_id>
+            <topic>camera/image_raw</topic>
+            <gz_frame_id>camera_link_optical</gz_frame_id>
         </sensor>
     </gazebo>

File: src/golftrolley/description/right_camera.xacro (robot description, xacro)
@@ -4,5 +4,5 @@
         <parent link="base_link"/>
         <child link="right_camera_link"/>
-        <origin xyz="0.0 0.0 0.46" rpy="0 0 0"/>
+        <origin xyz="0.0 0.0 0.7" rpy="0 0 0"/>
     </joint>
     <link name="right_camera_link">

File: src/golftrolley/description/robot.urdf.xacro (robot description, xacro)
@@ -6,6 +6,7 @@
     <!-- <xacro:include filename="gazebo_control.xacro" /> -->
     <xacro:include filename="lidar.xacro" />
-    <xacro:include filename="left_camera.xacro" />
-    <xacro:include filename="right_camera.xacro" />
+    <!-- <xacro:include filename="left_camera.xacro" />
+    <xacro:include filename="right_camera.xacro" /> -->
+    <xacro:include filename="camera.xacro" />
     <xacro:if value="$(arg use_ros2_control)">
         <xacro:include filename="ros2_control.xacro" />
